File: KiCad/SuperSimonPlayerController/USB-C.kicad_sch (KiCad schematic)
At the start: 5 parts

Commit message: Added tech notes to USB schematic
Other:
- note added: "3A PTC Fuse"
- note added: "5.1k pull-down resistors on CC1 and CC2 request 5V up to 3A from the USB host."
- note added: "TVS diodes protect devices from over voltage events e.g. static discharge."
Changed lines of the file:
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@@
+		)
+	)
+	(text "5.1k pull-down resistors on CC1 and CC2\nrequest 5V up to 3A from the USB host."
+		(exclude_from_sim no)
+		(at 89.408 127 0)
+		(effects
+			(font
+				(size 1.27 1.27)
+			)
+			(justify left)
+		)
+	)
+	(text "3A PTC Fuse"
+		(exclude_from_sim no)
+		(at 134.874 52.578 0)
+		(effects
+			(font
+				(size 1.27 1.27)
+			)
+		)
+	)
+	(text "TVS diodes protect devices from\nover voltage events e.g. static discharge."
+		(exclude_from_sim no)
+		(at 174.244 103.886 0)
+		(effects
+			(font
+				(size 1.27 1.27)
+			)
+			(justify left)
 		)
 	)
